File: TCC-PCB/TCC-PCB.kicad_sch (KiCad schematic)
At the start: 32 parts, among them SW1 SW_Push, U1 ATmega32U4-A, Y1 Crystal_GND24_Small

Commit message: changes
Parts:
- MX1, MX2, MX7, MX8: footprint (none) -> keebs:Mx_Alps_100
- MX3: renamed from MX5; footprint (none) -> keebs:Mx_Alps_100
- MX4: renamed from MX6; footprint (none) -> keebs:Mx_Alps_100
- MX5: renamed from MX3; footprint (none) -> keebs:Mx_Alps_100
- MX6: renamed from MX4; footprint (none) -> keebs:Mx_Alps_100
Connections:
- net COL0: no longer MX5.1 (COL)
- net COL1: now also MX5.1 (COL); no longer MX6.1 (COL)
- net COL2: now also MX6.1 (COL), U1.30 (PB6); no longer MX7.1 (COL)
- net COL3: now also MX7.1 (COL); no longer MX8.1 (COL)
- net ROW1: now also U1.26 (PD6); no longer U1.32 (PC7)
- new net COL4: MX8.1 (COL), U1.32 (PC7)
Other:
- moved on the sheet: D3, D4, D7, D8, MX5, MX6, MX7, MX8

Commit message: name change
Parts:
- MX1, MX2, MX3, MX4, MX5, MX6, MX7, MX8: footprint keebs:Mx_Alps_100 -> MX_Alps_Hybrid:MX-1U
- renumbered D3 to D2, D2 to D3, D7 to D6, D6 to D7
Connections:
- net COL1: now also MX3.1 (COL); no longer MX5.1 (COL)
- net COL2: now also MX4.1 (COL), MX5.1 (COL); no longer MX3.1 (COL), MX6.1 (COL)
- net COL3: now also MX6.1 (COL); no longer MX4.1 (COL)
- net at D2.2 (A): now also MX2.2 (ROW); no longer MX5.2 (ROW)
- net at MX7.2 (ROW): now also D7.2 (A); no longer D6.2 (A)
- net at MX3.2 (ROW): now also D3.2 (A); no longer D5.2 (A)
- net at MX6.2 (ROW): now also D6.2 (A); no longer D4.2 (A)
- net at MX4.2 (ROW): now also D4.2 (A); no longer D7.2 (A)
- new net: D5.2 (A), MX5.2 (ROW)
Other:
- note added: "MX1"
- note added: "MX2"
- note added: "MX3"
- note added: "MX4"
- note added: "MX5"
- note added: "MX6"
- note added: "MX7"
- note added: "MX8"

Commit message: updates and used footprints
Parts:
- MX1, MX2, MX3, MX4, MX5, MX6, MX7, MX8: footprint MX_Alps_Hybrid:MX-1U -> MX_Only:MXOnly-1U-Hotswap
Changed lines of the file:
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@@
       (effects (font (size 0.508 0.508)))
     )
-    (property "Footprint" "MX_Alps_Hybrid:MX-1U" (at 225.425 69.215 0)
+    (property "Footprint" "MX_Only:MXOnly-1U-Hotswap" (at 225.425 69.215 0)
       (effects (font (size 1.524 1.524)) hide)
     )
@@
       (effects (font (size 0.508 0.508)))
     )
-    (property "Footprint" "MX_Alps_Hybrid:MX-1U" (at 167.005 69.215 0)
+    (property "Footprint" "MX_Only:MXOnly-1U-Hotswap" (at 167.005 69.215 0)
       (effects (font (size 1.524 1.524)) hide)
     )
@@
       (effects (font (size 0.508 0.508)))
     )
-    (property "Footprint" "MX_Alps_Hybrid:MX-1U" (at 225.425 86.995 0)
+    (property "Footprint" "MX_Only:MXOnly-1U-Hotswap" (at 225.425 86.995 0)
       (effects (font (size 1.524 1.524)) hide)
     )
@@
       (effects (font (size 0.508 0.508)))
     )
-    (property "Footprint" "MX_Alps_Hybrid:MX-1U" (at 205.105 86.995 0)
+    (property "Footprint" "MX_Only:MXOnly-1U-Hotswap" (at 205.105 86.995 0)
       (effects (font (size 1.524 1.524)) hide)
     )
@@
       (effects (font (size 0.508 0.508)))
     )
-    (property "Footprint" "MX_Alps_Hybrid:MX-1U" (at 186.055 86.995 0)
+    (property "Footprint" "MX_Only:MXOnly-1U-Hotswap" (at 186.055 86.995 0)
       (effects (font (size 1.524 1.524)) hide)
     )
@@
       (effects (font (size 0.508 0.508)))
     )
-    (property "Footprint" "MX_Alps_Hybrid:MX-1U" (at 186.055 69.215 0)
+    (property "Footprint" "MX_Only:MXOnly-1U-Hotswap" (at 186.055 69.215 0)
       (effects (font (size 1.524 1.524)) hide)
     )
@@
       (effects (font (size 0.508 0.508)))
     )
-    (property "Footprint" "MX_Alps_Hybrid:MX-1U" (at 206.375 69.215 0)
+    (property "Footprint" "MX_Only:MXOnly-1U-Hotswap" (at 206.375 69.215 0)
       (effects (font (size 1.524 1.524)) hide)
     )
@@
       (effects (font (size 0.508 0.508)))
     )
-    (property "Footprint" "MX_Alps_Hybrid:MX-1U" (at 245.745 86.995 0)
-      (effects (font (size 1.524 1.524)) hide)
-    )
+    (property "Footprint" "MX_Only:MXOnly-1U-Hotswap" (at 245.745 86.995 0)
+      (effects (font (size 1.524 1.524)) hide)
+    )

Commit message: final changes
Parts:
- MX1, MX2, MX3, MX4, MX5, MX6, MX7, MX8: footprint MX_Only:MXOnly-1U-Hotswap -> MX_Only:MXOnly-1U
Connections:
- net ROW0: now also D1.1 (K), D3.1 (K), D5.1 (K), D7.1 (K), U1.26 (PD6); no longer U1.27 (PD7)
- net ROW1: now also D2.1 (K), D4.1 (K), D6.1 (K), D8.1 (K), U1.27 (PD7); no longer U1.26 (PD6)
Changed lines of the file:
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@@
+    (stroke (width 0) (type default))
+  )
+  (wire (pts (xy 88.9 86.36) (xy 92.71 86.36))
     (stroke (width 0) (type default))
   )
@@
   )
   (wire (pts (xy 144.78 27.94) (xy 151.13 27.94))
+    (stroke (width 0) (type default))
+  )
+  (wire (pts (xy 88.9 83.82) (xy 92.71 83.82))
     (stroke (width 0) (type default))
   )
@@
     )
   )
-  (global_label "ROW1" (shape output) (at 158.75 95.25 0) (fields_autoplaced)
+  (global_label "ROW0" (shape input) (at 92.71 83.82 0) (fields_autoplaced)
     (effects (font (size 1.27 1.27)) (justify left))
-    (property "Intersheetrefs" "${INTERSHEET_REFS}" (at 166.9172 95.25 0)
+    (property "Intersheetrefs" "${INTERSHEET_REFS}" (at 100.8772 83.82 0)
       (effects (font (size 1.27 1.27)) (justify left) hide)
     )
   )
-  (global_label "ROW0" (shape input) (at 88.9 86.36 0) (fields_autoplaced)
-    (effects (font (size 1.27 1.27)) (justify left))
-    (property "Intersheetrefs" "${INTERSHEET_REFS}" (at 97.0672 86.36 0)
-      (effects (font (size 1.27 1.27)) (justify left) hide)
+  (global_label "ROW1" (shape input) (at 166.37 95.25 180) (fields_autoplaced)
+    (effects (font (size 1.27 1.27)) (justify right))
+    (property "Intersheetrefs" "${INTERSHEET_REFS}" (at 158.2028 95.25 0)
+      (effects (font (size 1.27 1.27)) (justify right) hide)
     )
   )
@@
     )
   )
+  (global_label "ROW0" (shape input) (at 166.37 77.47 180) (fields_autoplaced)
+    (effects (font (size 1.27 1.27)) (justify right))
+    (property "Intersheetrefs" "${INTERSHEET_REFS}" (at 158.2028 77.47 0)
+      (effects (font (size 1.27 1.27)) (justify right) hide)
+    )
+  )
   (global_label "D-" (shape input) (at 115.57 30.48 0) (fields_autoplaced)
     (effects (font (size 1.27 1.27)) (justify left))
@@
     )
   )
-  (global_label "ROW1" (shape input) (at 88.9 83.82 0) (fields_autoplaced)
+  (global_label "ROW1" (shape input) (at 92.71 86.36 0) (fields_autoplaced)
     (effects (font (size 1.27 1.27)) (justify left))
-    (property "Intersheetrefs" "${INTERSHEET_REFS}" (at 97.0672 83.82 0)
-      (effects (font (size 1.27 1.27)) (justify left) hide)
-    )
-  )
-  (global_label "ROW0" (shape output) (at 158.75 77.47 0) (fields_autoplaced)
-    (effects (font (size 1.27 1.27)) (justify left))
-    (property "Intersheetrefs" "${INTERSHEET_REFS}" (at 166.9172 77.47 0)
+    (property "Intersheetrefs" "${INTERSHEET_REFS}" (at 100.8772 86.36 0)
       (effects (font (size 1.27 1.27)) (justify left) hide)
     )
@@
       (effects (font (size 0.508 0.508)))
     )
-    (property "Footprint" "MX_Only:MXOnly-1U-Hotswap" (at 225.425 69.215 0)
+    (property "Footprint" "MX_Only:MXOnly-1U" (at 225.425 69.215 0)
       (effects (font (size 1.524 1.524)) hide)
     )
@@
       (effects (font (size 0.508 0.508)))
     )
-    (property "Footprint" "MX_Only:MXOnly-1U-Hotswap" (at 167.005 69.215 0)
+    (property "Footprint" "MX_Only:MXOnly-1U" (at 167.005 69.215 0)
       (effects (font (size 1.524 1.524)) hide)
     )
@@
       (effects (font (size 0.508 0.508)))
     )
-    (property "Footprint" "MX_Only:MXOnly-1U-Hotswap" (at 225.425 86.995 0)
+    (property "Footprint" "MX_Only:MXOnly-1U" (at 225.425 86.995 0)
       (effects (font (size 1.524 1.524)) hide)
     )
@@
   )
   (symbol (lib_id "Device:D_Small") (at 194.31 92.71 90) (unit 1)
-    (in_bom yes) (on_board yes) (dnp no) (fields_autoplaced)
+    (in_bom yes) (on_board yes) (dnp no)
     (property "Reference" "D2" (at 196.85 92.075 90)
       (effects (font (size 1.27 1.27)) (justify right))
@@
       (effects (font (size 0.508 0.508)))
     )
-    (property "Footprint" "MX_Only:MXOnly-1U-Hotswap" (at 205.105 86.995 0)
+    (property "Footprint" "MX_Only:MXOnly-1U" (at 205.105 86.995 0)
       (effects (font (size 1.524 1.524)) hide)
     )
@@
       (effects (font (size 0.508 0.508)))
     )
-    (property "Footprint" "MX_Only:MXOnly-1U-Hotswap" (at 186.055 86.995 0)
+    (property "Footprint" "MX_Only:MXOnly-1U" (at 186.055 86.995 0)
       (effects (font (size 1.524 1.524)) hide)
     )
@@
       (effects (font (size 0.508 0.508)))
     )
-    (property "Footprint" "MX_Only:MXOnly-1U-Hotswap" (at 186.055 69.215 0)
+    (property "Footprint" "MX_Only:MXOnly-1U" (at 186.055 69.215 0)
       (effects (font (size 1.524 1.524)) hide)
     )
@@
       (effects (font (size 0.508 0.508)))
     )
-    (property "Footprint" "MX_Only:MXOnly-1U-Hotswap" (at 206.375 69.215 0)
+    (property "Footprint" "MX_Only:MXOnly-1U" (at 206.375 69.215 0)
       (effects (font (size 1.524 1.524)) hide)
     )
@@
       (effects (font (size 0.508 0.508)))
     )
-    (property "Footprint" "MX_Only:MXOnly-1U-Hotswap" (at 245.745 86.995 0)
-      (effects (font (size 1.524 1.524)) hide)
-    )
+    (property "Footprint" "MX_Only:MXOnly-1U" (at 245.745 86.995 0)
+      (effects (font (size 1.524 1.524)) hide)
+    )
